File: pcb/fab26_cablebot.kicad_pcb (KiCad board)
At the start: 2 copper layers, 66 x 45.2 mm, 28 parts, among them J1 LDR, J2 LDR, J3 9V BATTERY, J4 Neopixel continued, J5 MOTOR, J6 Servo, J8 BUZZER, SW1 ON/OFF, U1 XIAO-ESP32-C3-DIP, U2 5V REG, U3 Neopixel, U4 Grove I2C, U5 MotorDriver_BrushedDC_Toshiba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, U6 Grove I2C, U7 Grove Extra

Commit message: Finalize production version of PCB
Parts:
- added G***: LOGO, LOGO, F.Cu at (143.2, 98.0)
- added G***: LOGO, LOGO, B.Cu at (147.4, 91.7)
- moved U7 0.18 mm to (122.3, 84.2)
Other:
- board text added: "CABLEBOTTT"
