File: pcb/fab26_cablebot.kicad_sch (KiCad schematic)
At the start: 28 parts, among them J1 LDR, J2 LDR, J3 9V BATTERY, J4 Neopixel continued, J5 MOTOR, J6 Servo, J8 BUZZER, SW1 ON/OFF, U1 XIAO-ESP32-C3-DIP, U2 5V REG, U3 Neopixel, U4 Grove I2C, U5 MotorDriver_BrushedDC_Toshiba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, U6 Grove I2C, U7 Grove Extra

Commit message: Finalize production version of PCB
Parts:
- C2: value CP_Elec_100uF_Panasonic_EEE-FN1E101UL -> 100uF
- R4: value TBD - current sense (0.2, 0.5) -> 0.5R
Changed lines of the file:
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@@
 			)
 		)
-		(property "Value" "TBD - current sense (0.2, 0.5)"
+		(property "Value" "0.5R"
 			(at 184.15 54.61 90)
 			(show_name no)
@@
 			)
 		)
-		(property "Value" "CP_Elec_100uF_Panasonic_EEE-FN1E101UL"
+		(property "Value" "100uF"
 			(at 254 49.2124 0)
 			(show_name no)
